Commit message: remove joint limits (but not self-collisions)

File: models/gen3_7dof/urdf/GEN3_URDF_V12.urdf (robot description, URDF)
Before this commit: robot GEN3_URDF_V12, 9 links, 8 joints
Joints:
- joint Actuator1: limit effort=39 velocity=0.8727 -> (none)
- joint Actuator2: limit lower=-2.41 upper=2.41 effort=39 velocity=0.8727 -> (none)
- joint Actuator3: limit effort=39 velocity=0.8727 -> (none)
- joint Actuator4: limit lower=-2.66 upper=2.66 effort=39 velocity=0.8727 -> (none)
- joint Actuator5: limit effort=9 velocity=0.8727 -> (none)
- joint Actuator6: limit lower=-2.23 upper=2.23 effort=9 velocity=0.8727 -> (none)
- joint Actuator7: limit effort=9 velocity=0.8727 -> (none)
